Commit message: Punto 2a completato

File: ros2_iiwa/iiwa_description/urdf/iiwa.urdf.xacro (robot description, xacro)
@@ -5,4 +5,7 @@
     <color rgba="0.5 0.5 0.5 1.0"/>
   </material>
+  <material name="blue">
+    <color rgba="0.0 0.0 0.1 1.0"/>
+  </material>
   <link name="${prefix}iiwa_base" type="fixed"/>
   <joint name="${prefix}iiwa_root_joint" type="fixed">
@@ -173,37 +176,39 @@
 <parent link="${prefix}tool0"/>
 <child link="camera_link"/>
-<origin xyz="0.7 0 0.05" rpy="0 -1.57 0"/>
+<origin xyz="0.0 0 0.0" rpy="3.14 -1.57 0"/>
 </joint>
-  <link name="camera_link">
-<visual>
-<geometry>
-<box size="0.01 0.01 0.01"/>
-</geometry>
-<material name="red"/>
-</visual>
-<sensor name="iiwa_camera_sensor" type="camera">
-      <always_on>true</always_on>
-      <update_rate>30</update_rate>
-      <visualize>true</visualize>
-      <pose>0 0 0 0 0 0</pose>
-      <camera>
-        <horizontal_fov>1.57</horizontal_fov>
-        <image>
-          <width>1920</width>
-          <height>1080</height>
-          <format>R8G8B8</format>
-        </image>
-        <clip>
-          <near>0.1</near>
-          <far>100</far>
-        </clip>
-      </camera>
-      <plugin name="gz_camera_plugin" filename="gz-sim-camera-system">
-        <gz-sim-camera>
-          <topic>camera</topic>
-        </gz-sim-camera>
-      </plugin>
-    </sensor>
+<gazebo>
+	  <plugin filename="gz-sim-sensors-system"
+		name="gz::sim::systems::Sensors">
+		<render_engine>ogre2</render_engine>
+	</plugin>
+</gazebo>
+<link name="camera_link">
+  <visual>
+    <geometry>
+      <box size="0.02 0.02 0.02"/>
+    </geometry>
+      <material name="blue"/>
+  </visual>
 </link>
+<gazebo reference="camera_link">
+  <sensor name="camera0" type="camera">
+    <camera>
+      <horizontal_fov>1.047</horizontal_fov>
+      <image>
+        <width>340</width>
+        <height>200</height>
+      </image>
+      <clip>
+        <near>0.1</near>
+        <far>100</far>
+      </clip>
+    </camera>
+    <always_on>1</always_on>
+    <update_rate>30</update_rate>
+    <visualize>true</visualize>
+    <topic>camera</topic>
+  </sensor>
+</gazebo>
   <joint name="${prefix}joint_a1" type="revolute">
       <origin rpy="0 0 0" xyz="0 0 0"/>

Commit message: punto 2a sistemato

File: ros2_iiwa/iiwa_description/urdf/iiwa.urdf.xacro (robot description, xacro)
@@ -5,7 +5,4 @@
     <color rgba="0.5 0.5 0.5 1.0"/>
   </material>
-  <material name="blue">
-    <color rgba="0.0 0.0 0.1 1.0"/>
-  </material>
   <link name="${prefix}iiwa_base" type="fixed"/>
   <joint name="${prefix}iiwa_root_joint" type="fixed">
@@ -173,5 +170,5 @@
   </link>
   <link name="${prefix}tool0"/>
-  <joint name="camera_joint" type="fixed">
+<joint name="camera_joint" type="fixed">
 <parent link="${prefix}tool0"/>
 <child link="camera_link"/>

Commit message: punto 2c

File: ros2_iiwa/iiwa_description/urdf/iiwa.urdf.xacro (robot description, xacro)
@@ -170,4 +170,42 @@
   </link>
   <link name="${prefix}tool0"/>
+<joint name="camera_joint" type="fixed">
+<parent link="${prefix}tool0"/>
+<child link="camera_link"/>
+<origin xyz="0.0 0 0.0" rpy="3.14 -1.57 0"/>
+</joint>
+<gazebo>
+	  <plugin filename="gz-sim-sensors-system"
+		name="gz::sim::systems::Sensors">
+		<render_engine>ogre2</render_engine>
+	</plugin>
+</gazebo>
+<link name="camera_link">
+  <visual>
+    <geometry>
+      <box size="0.02 0.02 0.02"/>
+    </geometry>
+      <material name="blue"/>
+  </visual>
+</link>
+<gazebo reference="camera_link">
+  <sensor name="camera" type="camera">
+    <camera>
+      <horizontal_fov>1.047</horizontal_fov>
+      <image>
+        <width>340</width>
+        <height>200</height>
+      </image>
+      <clip>
+        <near>0.1</near>
+        <far>100</far>
+      </clip>
+    </camera>
+    <always_on>1</always_on>
+    <update_rate>30</update_rate>
+    <visualize>true</visualize>
+    <topic>camera</topic>
+  </sensor>
+</gazebo>
   <joint name="${prefix}joint_a1" type="revolute">
       <origin rpy="0 0 0" xyz="0 0 0"/>
